Commit message: navigation completed

File: urdf/gps.xacro (robot description, xacro)
@@ -12,4 +12,7 @@
             <color rgba="1 0 0 0.5"/>
         </material>
+        <gazebo reference="gps_link">
+          <material>Gazebo/Red</material>
+       </gazebo>
         <link name="gps_link">
             <visual>
@@ -37,8 +40,8 @@
             <plugin name="gps_controller" filename="libhector_gazebo_ros_gps.so">
                <updateRate>1000</updateRate>
-               <robotNamespace>robot</robotNamespace>
+               <robotNamespace>/</robotNamespace>
                <bodyName>gps_link</bodyName>
-               <topicName>fix</topicName>
-               <velocityTopicName>vel</velocityTopicName>
+               <topicName>robot/fix</topicName>
+               <velocityTopicName>robot/vel</velocityTopicName>
                <referenceLatitude>40.798824</referenceLatitude>
                <referenceLongitude>16.923127</referenceLongitude>

File: urdf/imu.xacro (robot description, xacro)
@@ -8,18 +8,24 @@
             <origin rpy="0 0 0" xyz="${x} ${y} ${z}"/>
         </joint>
-      <gazebo>
-        <plugin name="imu_controller" filename="libhector_gazebo_ros_imu.so">
-         <robotNamespace>robot</robotNamespace>
-         <updateRate>50.0</updateRate>
-         <bodyName>imu_link</bodyName>
-         <topicName>imu/data</topicName>
-         <accelDrift>0.005 0.005 0.005</accelDrift>
-         <accelGaussianNoise>0.005 0.005 0.005</accelGaussianNoise>
-         <rateDrift>0.005 0.005 0.005 </rateDrift>
-         <rateGaussianNoise>0.005 0.005 0.005 </rateGaussianNoise>
-         <headingDrift>0.005</headingDrift>
-         <headingGaussianNoise>0.005</headingGaussianNoise>
-        </plugin>
-      </gazebo>
+        <gazebo reference="imu_link">
+           <gravity>true</gravity>
+           <sensor name="imu_sensor" type="imu">
+             <always_on>true</always_on>
+             <update_rate>50</update_rate>
+             <visualize>true</visualize>
+             <topic>robot/imu</topic>
+             <plugin filename="libgazebo_ros_imu_sensor.so" name="imu_plugin">
+              <topicName>robot/imu</topicName>
+              <bodyName>imu_link</bodyName>
+              <updateRateHZ>10.0</updateRateHZ>
+              <gaussianNoise>0.0</gaussianNoise>
+              <xyzOffset>0 0 0</xyzOffset>
+              <rpyOffset>0 0 0</rpyOffset>
+              <frameName>imu_link</frameName>
+              <initialOrientationAsReference>false</initialOrientationAsReference>
+             </plugin>
+             <pose>0 0 0 0 0 0</pose>
+           </sensor>
+        </gazebo>
     </xacro:macro>
 </robot>

File: urdf/laser.xacro (robot description, xacro)
@@ -12,4 +12,7 @@
             <color rgba="1 0.51 0 0.5"/>
         </material>
+       <gazebo reference="laser_link">
+          <material>Gazebo/Orange</material>
+       </gazebo>
         <link name="laser_link">
             <visual>
@@ -37,6 +40,6 @@
             <sensor type="ray" name="head_hokuyo_sensor">
                 <pose>0 0 0 0 0 0</pose>
-                <visualize>false</visualize>
-                <update_rate>40</update_rate>
+                <visualize>true</visualize>
+                <update_rate>50</update_rate>
                 <ray>
                     <scan>

File: urdf/robot.xacro (robot description, xacro)
@@ -10,5 +10,5 @@
     <!-- heros base-->
     <xacro:innok_heros front_kind='$(arg front_kind)' wheel_kind='$(arg wheel_kind)'/>
-    <xacro:robot_laser x="0.82" y="0" z="0.1" laser_size="0.1"/>
+    <xacro:robot_laser x="0.85" y="0" z="0" laser_size="0.1"/>
     <xacro:plow x="-1" y="0" z="0"/>
     <xacro:robot_gps x="0" y="0" z="0.1" gps_size="0.1" />
